File: kicad/four_way_rotator.kicad_pcb (KiCad board)
At the start: 4 copper layers, 140.7 x 54 mm, 57 parts, among them J1 USB_B_Micro, J2 Peripheral, J3 Barrel_Jack_Switch, J4 NeoPixels, J5 Motor, J6 Motor, SW1 BOOT, SW2 RESET, U1 TPS563200, U2 TPS5403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

Commit message: Fixed feedback node routing
Routing:
- net Net-(U1-VFB): track 10.3 -> 15.4 mm, vias 0 -> 2
Changed lines of the file:
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@@
-	)
-	(segment
-		(start 105.481127 85.2249)
-		(end 105.481127 85.464576)
-		(width 0.25)
-		(layer "F.Cu")
-		(net 18)
 	)
 	(segment
@@
 	)
 	(segment
-		(start 104.945703 86)
-		(end 103.631127 86)
-		(width 0.25)
-		(layer "F.Cu")
-		(net 18)
-	)
-	(segment
-		(start 106.081127 81.837501)
-		(end 106.081127 84.6249)
-		(width 0.25)
-		(layer "F.Cu")
-		(net 18)
-	)
-	(segment
-		(start 103.631127 86)
-		(end 102.831127 86.8)
-		(width 0.25)
-		(layer "F.Cu")
-		(net 18)
-	)
-	(segment
-		(start 106.081127 84.6249)
-		(end 105.481127 85.2249)
-		(width 0.25)
-		(layer "F.Cu")
-		(net 18)
-	)
-	(segment
-		(start 105.481127 85.464576)
-		(end 104.945703 86)
-		(width 0.25)
+		(start 101.5 86.5)
+		(end 102.531127 86.5)
+		(width 0.2)
 		(layer "F.Cu")
 		(net 18)
@@
 	(segment
 		(start 104.881127 81.3)
-		(end 105.543626 81.3)
-		(width 0.25)
+		(end 104.8 81.3)
+		(width 0.2)
 		(layer "F.Cu")
 		(net 18)
 	)
 	(segment
-		(start 105.543626 81.3)
-		(end 106.081127 81.837501)
-		(width 0.25)
+		(start 104.8 81.3)
+		(end 104 80.5)
+		(width 0.2)
 		(layer "F.Cu")
 		(net 18)
 	)
+	(segment
+		(start 102.531127 86.5)
+		(end 102.831127 86.8)
+		(width 0.2)
+		(layer "F.Cu")
+		(net 18)
+	)
+	(via
+		(at 104 80.5)
+		(size 0.6)
+		(drill 0.3)
+		(layers "F.Cu" "B.Cu")
+		(net 18)
+	)
+	(via
+		(at 101.5 86.5)
+		(size 0.6)
+		(drill 0.3)
+		(layers "F.Cu" "B.Cu")
+		(net 18)
+	)
+	(segment
+		(start 99.712902 84.712902)
+		(end 101.5 86.5)
+		(width 0.2)
+		(layer "B.Cu")
+		(net 18)
+	)
+	(segment
+		(start 99.712902 81.287098)
+		(end 99.712902 84.712902)
+		(width 0.2)
+		(layer "B.Cu")
+		(net 18)
+	)
+	(segment
+		(start 103.5 80)
+		(end 101 80)
+		(width 0.2)
+		(layer "B.Cu")
+		(net 18)
+	)
+	(segment
+		(start 104 80.5)
+		(end 103.5 80)
+		(width 0.2)
+		(layer "B.Cu")
+		(net 18)
+	)
+	(segment
+		(start 101 80)
+		(end 100 81)
+		(width 0.2)
+		(layer "B.Cu")
+		(net 18)
+	)
+	(segment
+		(start 100 81)
+		(end 99.712902 81.287098)
+		(width 0.2)
+		(layer "B.Cu")
+		(net 18)
+	)
